Commit message: update packages

File: install/rmitbot_description/share/rmitbot_description/urdf/rmitbot.urdf.xacro (robot description, xacro)
@@ -5,6 +5,6 @@
 <robot name="rmitbot"
     xmlns:xacro="http://ros.org/wiki/xacro">
-    <!-- Include Gazebo Parameters -->
     <xacro:include filename="$(find rmitbot_description)/urdf/rmitbot_platform.xacro" />
     <xacro:include filename="$(find rmitbot_description)/urdf/rmitbot_gazebo.xacro" />
+    <xacro:include filename="$(find rmitbot_description)/urdf/rmitbot_ros2_control.xacro" />
 </robot>

File: install/rmitbot_description/share/rmitbot_description/urdf/rmitbot_gazebo.xacro (robot description, xacro)
@@ -1,40 +1,63 @@
 <?xml version="1.0"?>
 <!-- Gazebo file contains information regarding the lnks's physics (e.g., friction, stiffness, damping) -->
-<robot name="rmitbot" xmlns:xacro="http://ros.org/wiki/xacro">
+<robot name="rmitbot" xmlns:xacro="http://ros.org/wiki/xacro" xmlns:gz="http://gazebosim.org/schema">
   <!-- Wheels -->
-  <gazebo reference="wheel_left_link">
-    <mu1>1000000000000000.0</mu1>
-    <mu2>1000000000000000.0</mu2>
-    <kp>1000000000000.0</kp>
-    <kd>10.0</kd>
-    <minDepth>0.001</minDepth>
-    <maxVel>0.1</maxVel>
-    <fdir1>1 0 0</fdir1>
+     <!-- To emulate Mecanum wheels in Gazebo with spherical collisions it
+  requires a custom friction model so the vehicle can strafe left to right -->
+  <gazebo reference='front_left_wheel'>
+    <collision>
+      <surface>
+        <friction>
+          <ode>
+            <mu>1.0</mu>
+            <mu2>0.0</mu2>
+            <!-- <fdir1 gz:expressed_in="base_link">1 -1 0</fdir1> -->
+            <fdir1 gz:expressed_in="base_footprint">1 -1 0</fdir1>
+          </ode>
+        </friction>
+      </surface>
+    </collision>
   </gazebo>
-  <gazebo reference="wheel_right_link">
-    <mu1>1000000000000000.0</mu1>
-    <mu2>1000000000000000.0</mu2>
-    <kp>1000000000000.0</kp>
-    <kd>10.0</kd>
-    <minDepth>0.001</minDepth>
-    <maxVel>0.1</maxVel>
-    <fdir1>1 0 0</fdir1>
+  <gazebo reference='front_right_wheel'>
+    <collision>
+      <surface>
+        <friction>
+          <ode>
+            <mu>1.0</mu>
+            <mu2>0.0</mu2>
+            <!-- <fdir1 gz:expressed_in="base_link">1 1 0</fdir1> -->
+            <fdir1 gz:expressed_in="base_footprint">1 1 0</fdir1>
+          </ode>
+        </friction>
+      </surface>
+    </collision>
   </gazebo>
-  <!-- Caster Wheels -->
-  <gazebo reference="caster_rear_link">
-    <mu1>0.1</mu1>
-    <mu2>0.1</mu2>
-    <kp>1000000.0</kp>
-    <kd>100.0</kd>
-    <minDepth>0.001</minDepth>
-    <maxVel>1.0</maxVel>
+  <gazebo reference='rear_left_wheel'>
+    <collision>
+      <surface>
+        <friction>
+          <ode>
+            <mu>1.0</mu>
+            <mu2>0.0</mu2>
+            <!-- <fdir1 gz:expressed_in="base_link">1 1 0</fdir1> -->
+            <fdir1 gz:expressed_in="base_footprint">1 1 0</fdir1>
+          </ode>
+        </friction>
+      </surface>
+    </collision>
   </gazebo>
-  <gazebo reference="caster_front_link">
-    <mu1>0.1</mu1>
-    <mu2>0.1</mu2>
-    <kp>1000000.0</kp>
-    <kd>100.0</kd>
-    <minDepth>0.001</minDepth>
-    <maxVel>1.0</maxVel>
+  <gazebo reference='rear_right_wheel'>
+    <collision>
+      <surface>
+        <friction>
+          <ode>
+            <mu>1.0</mu>
+            <mu2>0.0</mu2>
+            <!-- <fdir1 gz:expressed_in="base_link">1 -1 0</fdir1> -->
+            <fdir1 gz:expressed_in="base_footprint">1 -1 0</fdir1>
+          </ode>
+        </friction>
+      </surface>
+    </collision>
   </gazebo>
 </robot>

File: install/rmitbot_description/share/rmitbot_description/urdf/rmitbot_platform.xacro (robot description, xacro)
@@ -1,132 +1,189 @@
 <?xml version="1.0"?>
-<!-- This file contains the urdf of the base platform -->
-<!-- Description of the robot in URDF format -->
-<!-- Each link must have at least visual for rivz -->
-<!-- Each link must have inertia and collision for gazebo -->
-<robot name="rmitbot" xmlns:xacro="http://ros.org/wiki/xacro">
-    <link name="base_footprint"/>
-    <link name="base_link">
-        <inertial>
-            <origin xyz="0 0 0.04" rpy="0.0 0.25 0.3" />
-            <mass value="8.2573504e-01"/>
-            <inertia ixx="2.2124416e-02" ixy="-1.2294101e-04" ixz="3.4938785e-04" iyy="2.1193702e-02" iyz="-5.0120904e-05" izz="2.0064271e-02" />
-        </inertial>
-        <visual>
-            <origin xyz="0 0 0" rpy="0 0 0" />
-            <geometry>
-                <mesh filename="package://rmitbot_description/meshes/base_link.STL" />
-            </geometry>
-        </visual>
-        <collision>
-            <origin xyz="0 0 0" rpy="0 0 0" />
-            <geometry>
-                <mesh filename="package://rmitbot_description/meshes/base_link.STL" />
-            </geometry>
-        </collision>
-    </link>
-    <joint name="base_joint" type="fixed">
-        <parent link="base_footprint"/>
-        <child link="base_link" />
-        <origin xyz="0 0 0.033" rpy="0 0 0"/>
-    </joint>
-    <link name="wheel_right_link">
-        <inertial>
-            <origin xyz="0 -0.014 0" rpy="0 0 0" />
-            <mass value="0.0530086090966721" />
-            <inertia ixx="1.88176298336665E-05" ixy="-4.8444933029987E-10" ixz="1.88163708851143E-08" iyy="3.11510738647764E-05" iyz="-6.93560663069607E-11" izz="1.8801969558182E-05" />
-        </inertial>
-        <visual>
-            <origin xyz="0 0 0" rpy="1.57 0 0" />
-            <geometry>
-                <mesh filename="package://rmitbot_description/meshes/wheel_right_link.STL" />
-            </geometry>
-        </visual>
-        <collision>
-            <origin xyz="0 -0.015 0" rpy="1.57 0 0" />
-            <geometry>
-                <sphere radius="0.033"/>
-            </geometry>
-        </collision>
-    </link>
-    <joint name="wheel_right_joint" type="continuous">
-        <origin xyz="0 -0.0701101849418637 0" rpy="0 0 0" />
-        <parent link="base_link" />
-        <child link="wheel_right_link" />
-        <axis xyz="0 1 0" />
-    </joint>
-    <link name="wheel_left_link">
-        <inertial>
-            <origin xyz="0 0.014 0" rpy="0 0 0" />
-            <mass value="0.0530086043217644" />
-            <inertia ixx="1.8792911368909E-05" ixy="3.31256392204584E-10" ixz="-1.14082001662767E-08" iyy="3.11510738759073E-05" iyz="-3.60499245082192E-10" izz="1.88266886146847E-05" />
-        </inertial>
-        <visual>
-            <origin xyz="0 0 0" rpy="-1.57 0 0" />
-            <geometry>
-                <mesh filename="package://rmitbot_description/meshes/wheel_left_link.STL" />
-            </geometry>
-        </visual>
-        <collision>
-            <origin xyz="0 0.015 0" rpy="-1.57 0 0" />
-            <geometry>
-                <sphere radius="0.033"/>
-            </geometry>
-        </collision>
-    </link>
-    <joint name="wheel_left_joint" type="continuous">
-        <origin xyz="0 0.0701101849418642 0" rpy="0 0 0" />
-        <parent link="base_link" />
-        <child link="wheel_left_link" />
-        <axis xyz="0 1 0" />
-    </joint>
-    <link name="caster_front_link">
-        <inertial>
-            <origin xyz="3.89968128948481E-07 2.40073004698083E-07 0.00219173397061506" rpy="0 0 0" />
-            <mass value="1.44379265037903E-06" />
-            <inertia ixx="7.23075276010246E-11" ixy="-6.10956883467859E-16" ixz="2.22849693525031E-15" iyy="3.8713793085917E-11" iyz="2.93909858781952E-15" izz="1.00967486676306E-10" />
-        </inertial>
-        <visual>
-            <origin xyz="0 0 0" rpy="0 0 0" />
-            <geometry>
-                <mesh filename="package://rmitbot_description/meshes/caster_front_link.STL" />
-            </geometry>
-        </visual>
-        <collision>
-            <origin xyz="0 0 0" rpy="0 0 0" />
-            <geometry>
-                <sphere radius="0.005"/>
-            </geometry>
-        </collision>
-    </link>
-    <joint name="caster_front_joint" type="fixed">
-        <origin xyz="0.04755 0 -0.0275" rpy="0 0 0" />
-        <parent link="base_link" />
-        <child link="caster_front_link" />
-        <axis xyz="0 0 0" />
-    </joint>
-    <link name="caster_rear_link">
-        <inertial>
-            <origin xyz="3.8996812895542E-07 2.40073004698083E-07 0.00219173397061509" rpy="0 0 0" />
-            <mass value="1.44379265037902E-06" />
-            <inertia ixx="7.23075276010246E-11" ixy="-6.10956872363424E-16" ixz="2.22849693527207E-15" iyy="3.87137930859167E-11" iyz="2.939098587861E-15" izz="1.00967486676306E-10" />
-        </inertial>
-        <visual>
-            <origin xyz="0 0 0" rpy="0 0 0" />
-            <geometry>
-                <mesh filename="package://rmitbot_description/meshes/caster_rear_link.STL" />
-            </geometry>
-        </visual>
-        <collision>
-            <origin xyz="0 0 0" rpy="0 0 0" />
-            <geometry>
-                <sphere radius="0.005"/>
-            </geometry>
-        </collision>
-    </link>
-    <joint name="caster_rear_joint" type="fixed">
-        <origin xyz="-0.04755 0 -0.0275" rpy="0 0 0" />
-        <parent link="base_link" />
-        <child link="caster_rear_link" />
-        <axis xyz="0 0 0" />
-    </joint>
+<robot name="rmitbot" xmlns:xacro="http://www.ros.org/wiki/xacro" xmlns:gz="http://gazebosim.org/schema">
+  <material name="orange">
+    <color rgba="0.8 0.4 0.0 1.0" />
+  </material>
+  <material name="black">
+    <color rgba="0.5 0.5 0.5 1.0" />
+  </material>
+  <material name="white">
+    <color rgba="1 1 1 1.0" />
+  </material>
+  <link name="base_footprint" />
+  <joint name="base_joint" type="fixed">
+    <parent link="base_footprint" />
+    <child link="base_link" />
+    <origin xyz="0 0 0.05" rpy="0 0 0" />
+  </joint>
+  <!-- Base Link -->
+  <link name="base_link">
+    <collision>
+      <origin xyz="0 0 0.05" rpy="0 0 0" />
+      <geometry>
+         <box size=".28 .3 0.1" />
+      </geometry>
+    </collision>
+    <visual>
+      <origin xyz="0 0 0.05" rpy="0 0 0" />
+      <geometry>
+         <box size=".28 .3 0.1" />
+      </geometry>
+      <material name="orange" />
+    </visual>
+    <inertial>
+      <origin xyz="0 0 0.5" rpy="0 0 0" />
+      <mass value="1.5" />
+      <inertia
+        ixx="0.13"
+        ixy="0.0"
+        ixz="0.0"
+        iyy="0.42"
+        iyz="0.0"
+        izz="0.48" />
+    </inertial>
+  </link>
+  <!-- front left wheel -->
+  <joint name="front_left_wheel_joint" type="continuous">
+    <origin xyz="0.14 0.15 0" rpy="-${pi/2} 0 0" />
+    <parent link="base_link" />
+    <child link="front_left_wheel" />
+    <axis xyz="0 0 1" />
+    <dynamics damping="0.2" />
+  </joint>
+  <link name="front_left_wheel">
+    <collision>
+      <!-- <origin xyz="0 0 .06" rpy="0 0 0" /> -->
+      <origin xyz="0 0 .025" rpy="0 0 0" />
+      <geometry>
+        <sphere radius="0.05" />
+      </geometry>
+    </collision>
+    <visual>
+      <!-- <origin xyz="0 0 .06" rpy="0 0 0" /> -->
+      <origin xyz="0 0 .025" rpy="0 0 0" />
+      <geometry>
+        <!-- <sphere radius="0.3" /> -->
+        <cylinder radius="0.05" length="0.05" />
+      </geometry>
+      <material name="black" />
+    </visual>
+    <inertial>
+      <!-- <origin xyz="0 0 .06" rpy="0 0 0" /> -->
+       <origin xyz="0 0 .025" rpy="0 0 0" />
+      <mass value="0.5" />
+      <inertia ixx="0.0025"
+        ixy="0.0"
+        ixz="0.0"
+        iyy="0.0025"
+        iyz="0.0"
+        izz="0.0020" />
+    </inertial>
+  </link>
+  <!-- front right wheel -->
+  <joint name="front_right_wheel_joint" type="continuous">
+    <origin xyz="0.14 -0.15 0." rpy="-${pi/2} 0 0" />
+    <parent link="base_link" />
+    <child link="front_right_wheel" />
+    <axis xyz="0 0 1" />
+    <dynamics damping="0.2" />
+  </joint>
+  <link name="front_right_wheel">
+    <collision>
+      <!-- <origin xyz="0 0 -.06" rpy="0 0 0" /> -->
+      <origin xyz="0 0 -.025" rpy="0 0 0" />
+      <geometry>
+        <sphere radius="0.05" />
+      </geometry>
+    </collision>
+    <visual>
+      <origin xyz="0 0 -.025" rpy="0 0 0" />
+      <geometry>
+        <cylinder radius="0.05" length="0.05" />
+      </geometry>
+      <material name="black" />
+    </visual>
+    <inertial>
+      <!-- <origin xyz="0 0 -.06" rpy="0 0 0" /> -->
+      <origin xyz="0 0 -.025" rpy="0 0 0" />
+      <mass value=".5" />
+      <inertia ixx="0.0025"
+        ixy="0.0"
+        ixz="0.0"
+        iyy="0.0025"
+        iyz="0.0"
+        izz="0.0020" />
+    </inertial>
+  </link>
+  <!-- rear left wheel -->
+  <joint name="rear_left_wheel_joint" type="continuous">
+    <origin xyz="-0.14 0.15 0." rpy="-${pi/2} 0 0" />
+    <parent link="base_link" />
+    <child link="rear_left_wheel" />
+    <axis xyz="0 0 1" />
+    <dynamics damping="0.2" />
+  </joint>
+  <link name="rear_left_wheel">
+    <collision>
+      <!-- <origin xyz="0 0 .06" rpy="0 0 0" /> -->
+       <origin xyz="0 0 .025" rpy="0 0 0" />
+      <geometry>
+        <sphere radius="0.05" />
+      </geometry>
+    </collision>
+    <visual>
+      <!-- <origin xyz="0 0 .06" rpy="0 0 0" /> -->
+       <origin xyz="0 0 .025" rpy="0 0 0" />
+      <geometry>
+        <cylinder radius="0.05" length="0.05" />
+      </geometry>
+      <material name="black" />
+    </visual>
+    <inertial>
+      <!-- <origin xyz="0 0 .06" rpy="0 0 0" /> -->
+       <origin xyz="0 0 .025" rpy="0 0 0" />
+      <mass value="0.5" />
+      <inertia ixx="0.0025"
+        ixy="0.0"
+        ixz="0.0"
+        iyy="0.0025"
+        iyz="0.0"
+        izz="0.0020" />
+    </inertial>
+  </link>
+  <!-- rear right wheel -->
+  <joint name="rear_right_wheel_joint" type="continuous">
+    <origin xyz="-0.14 -0.15 0." rpy="-${pi/2} 0 0" />
+    <parent link="base_link" />
+    <child link="rear_right_wheel" />
+    <axis xyz="0 0 1" />
+    <dynamics damping="0.2" />
+  </joint>
+  <link name="rear_right_wheel">
+    <collision>
+      <!-- <origin xyz="0 0 -.06" rpy="0 0 0" /> -->
+       <origin xyz="0 0 -.025" rpy="0 0 0" />
+      <geometry>
+        <sphere radius="0.05" />
+      </geometry>
+    </collision>
+    <visual>
+      <!-- <origin xyz="0 0 -.06" rpy="0 0 0" /> -->
+       <origin xyz="0 0 -.025" rpy="0 0 0" />
+      <geometry>
+        <cylinder radius="0.05" length="0.05" />
+      </geometry>
+      <material name="black" />
+    </visual>
+    <inertial>
+      <!-- <origin xyz="0 0 -.06" rpy="0 0 0" /> -->
+       <origin xyz="0 0 -.025" rpy="0 0 0" />
+      <mass value="0.5" />
+      <inertia ixx="0.0025"
+        ixy="0.0"
+        ixz="0.0"
+        iyy="0.0025"
+        iyz="0.0"
+        izz="0.0020" />
+    </inertial>
+  </link>
 </robot>

File: src/rmitbot_description/urdf/rmitbot_gazebo.xacro (robot description, xacro)
@@ -1,40 +1,63 @@
 <?xml version="1.0"?>
 <!-- Gazebo file contains information regarding the lnks's physics (e.g., friction, stiffness, damping) -->
-<robot name="rmitbot" xmlns:xacro="http://ros.org/wiki/xacro">
+<robot name="rmitbot" xmlns:xacro="http://ros.org/wiki/xacro" xmlns:gz="http://gazebosim.org/schema">
   <!-- Wheels -->
-  <gazebo reference="wheel_left_link">
-    <mu1>1000000000000000.0</mu1>
-    <mu2>1000000000000000.0</mu2>
-    <kp>1000000000000.0</kp>
-    <kd>10.0</kd>
-    <minDepth>0.001</minDepth>
-    <maxVel>0.1</maxVel>
-    <fdir1>1 0 0</fdir1>
+     <!-- To emulate Mecanum wheels in Gazebo with spherical collisions it
+  requires a custom friction model so the vehicle can strafe left to right -->
+  <gazebo reference='front_left_wheel'>
+    <collision>
+      <surface>
+        <friction>
+          <ode>
+            <mu>1.0</mu>
+            <mu2>0.0</mu2>
+            <!-- <fdir1 gz:expressed_in="base_link">1 -1 0</fdir1> -->
+            <fdir1 gz:expressed_in="base_footprint">1 -1 0</fdir1>
+          </ode>
+        </friction>
+      </surface>
+    </collision>
   </gazebo>
-  <gazebo reference="wheel_right_link">
-    <mu1>1000000000000000.0</mu1>
-    <mu2>1000000000000000.0</mu2>
-    <kp>1000000000000.0</kp>
-    <kd>10.0</kd>
-    <minDepth>0.001</minDepth>
-    <maxVel>0.1</maxVel>
-    <fdir1>1 0 0</fdir1>
+  <gazebo reference='front_right_wheel'>
+    <collision>
+      <surface>
+        <friction>
+          <ode>
+            <mu>1.0</mu>
+            <mu2>0.0</mu2>
+            <!-- <fdir1 gz:expressed_in="base_link">1 1 0</fdir1> -->
+            <fdir1 gz:expressed_in="base_footprint">1 1 0</fdir1>
+          </ode>
+        </friction>
+      </surface>
+    </collision>
   </gazebo>
-  <!-- Caster Wheels -->
-  <gazebo reference="caster_rear_link">
-    <mu1>0.1</mu1>
-    <mu2>0.1</mu2>
-    <kp>1000000.0</kp>
-    <kd>100.0</kd>
-    <minDepth>0.001</minDepth>
-    <maxVel>1.0</maxVel>
+  <gazebo reference='rear_left_wheel'>
+    <collision>
+      <surface>
+        <friction>
+          <ode>
+            <mu>1.0</mu>
+            <mu2>0.0</mu2>
+            <!-- <fdir1 gz:expressed_in="base_link">1 1 0</fdir1> -->
+            <fdir1 gz:expressed_in="base_footprint">1 1 0</fdir1>
+          </ode>
+        </friction>
+      </surface>
+    </collision>
   </gazebo>
-  <gazebo reference="caster_front_link">
-    <mu1>0.1</mu1>
-    <mu2>0.1</mu2>
-    <kp>1000000.0</kp>
-    <kd>100.0</kd>
-    <minDepth>0.001</minDepth>
-    <maxVel>1.0</maxVel>
+  <gazebo reference='rear_right_wheel'>
+    <collision>
+      <surface>
+        <friction>
+          <ode>
+            <mu>1.0</mu>
+            <mu2>0.0</mu2>
+            <!-- <fdir1 gz:expressed_in="base_link">1 -1 0</fdir1> -->
+            <fdir1 gz:expressed_in="base_footprint">1 -1 0</fdir1>
+          </ode>
+        </friction>
+      </surface>
+    </collision>
   </gazebo>
 </robot>
